File: cable_breakout/cable_breakout.sch (KiCad schematic (older format))
At the start: 35 parts, among them J1 Bergstak 20P female 3.7mm, J10 Conn_Coaxial_Power, J11 Conn_Coaxial_Power, J12 Conn_Coaxial_Power, J13 Conn_Coaxial_Power, J14 Conn_Coaxial_Power, J15 Conn_Coaxial_Power, J16 Conn_Coaxial_Power, J17 Conn_Coaxial_Power, J18 Conn_Coaxial_Power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

Commit message: Reorg boards into subdirs
Parts:
- gave numbers to parts that had none: 1
Changed lines of the file:
@@
 $EndComp
 $Comp
-L TEST TP?
+L TEST TP8
 U 1 1 5B38DE8E
 P 8500 2900
-F 0 "TP?" H 8500 3200 50  0000 C BNN
+F 0 "TP8" H 8500 3200 50  0000 C BNN
 F 1 "TEST" H 8500 3150 50  0000 C CNN
 F 2 "footprints:patch_pad" H 8500 2900 50  0001 C CNN
