File: cable_breakout/cable_breakout.kicad_pcb (KiCad board)
At the start: 2 copper layers, 45 x 50 mm, 38 parts, among them J1 Bergstak 20P female 3.7mm, J10 Conn_Coaxial_Power, J11 Conn_Coaxial_Power, J12 Conn_Coaxial_Power, J13 Conn_Coaxial_Power, J14 Conn_Coaxial_Power, J15 Conn_Coaxial_Power, J16 Conn_Coaxial_Power, J17 Conn_Coaxial_Power, J18 Conn_Coaxial_Power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

Commit message: Do proper pretty breakout gerber export
Other:
- board text added: "cable breakout board Project 002 v0.1"
Changed lines of the file:
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@@
-(kicad_pcb (version 4) (host pcbnew 4.0.7)
+(kicad_pcb (version 20171130) (host pcbnew "(5.0.1)")
   (general
-    (links 178)
-    (no_connects 4)
-    (area 89.650001 82.3 180.000001 145.200001)
     (thickness 1.6)
-    (drawings 68)
+    (drawings 69)
     (tracks 327)
     (zones 0)
@@
   )
   (setup
-    (last_trace_width 0.508)
+    (last_trace_width 0.15)
     (user_trace_width 0.1524)
     (user_trace_width 0.19)
@@
     (pad_drill 4)
     (pad_to_mask_clearance 0.06)
+    (solder_mask_min_width 0.25)
     (aux_axis_origin 0 0)
     (visible_elements FFFFFF7F)
@@
       (layerselection 0x010fc_80000001)
       (usegerberextensions true)
-      (excludeedgelayer true)
+      (usegerberattributes false)
+      (usegerberadvancedattributes false)
+      (creategerberjobfile false)
+      (excludeedgelayer false)
       (linewidth 0.100000)
       (plotframeref false)
@@
       (hpglpennumber 1)
       (hpglpenspeed 20)
-      (hpglpendiameter 15)
-      (hpglpenoverlay 2)
+      (hpglpendiameter 15.000000)
       (psnegative false)
       (psa4output false)
@@
       (drillshape 0)
       (scaleselection 1)
-      (outputdirectory gerber))
+      (outputdirectory "gerber"))
   )
   (net 0 "")
@@
       (net 2 VSSA))
   )
-  (gr_text COM (at 151.75 95.05 360) (layer B.SilkS)
+  (gr_text "cable breakout board\nProject 002\nv0.1" (at 113.3 128.3 90) (layer F.SilkS)
+    (effects (font (size 1.2 1.2) (thickness 0.24)) (justify left))
+  )
+  (gr_text COM (at 151.75 95.05) (layer B.SilkS)
     (effects (font (size 1 1) (thickness 0.2)) (justify mirror))
   )
